File: Button_And_Buzzer.kicad_sch (KiCad schematic)
At the start: 26 parts, among them Q3 S8050, SW3 SW_Push_Dual, SW4 SW_Push_Dual, SW5 SW_Push_Dual, SW6 SW_Push_Dual, SW7 SW_Push_Dual

Commit message: 2026 08 24 画图完成，准备生产
Parts:
- removed BZ1: Buzzer, Buzzer_Beeper:Buzzer_15x7.5RM7.6, symbol Device:Buzzer
- removed SW3, SW4, SW5, SW6, SW7: SW_Push_Dual, symbol Switch:SW_Push_Dual
- added BUZZER1: FST-5020, UPT:BUZ-SMD_FST-5020, symbol UPT:FST-5020
- added SW3, SW4, SW5, SW6, SW7: SW_Push_Dual, UPT:SW-TH_4P-L6.0-W6.0-P4.50-LS6.5, symbol UPT:SW_Push_Dual
- D16: footprint Diode_THT:D_DO-35_SOD27_P7.62mm_Horizontal -> Diode_SMD:D_SOD-123
- Q3: footprint Package_TO_SOT_THT:TO-92_Inline -> Package_TO_SOT_SMD:SOT-23_Handsoldering
Connections:
- net BUTTON_3V3: now also BUZZER1.1 (+)
- net GND: now also SW3.3, SW3.4, SW4.3, SW4.4, SW5.3, SW5.4, SW6.3, SW6.4, SW7.3, SW7.4
- net at R81.2, R82.1: now also SW3.1, SW3.2
- net at R83.2, R84.1: now also SW4.1, SW4.2
- net at R87.2, R88.1: now also SW6.1, SW6.2
- net at R89.2, R90.1: now also SW7.1, SW7.2
- net at R85.2, R86.1: now also SW5.1, SW5.2
- net at Q3.3 (C): now also BUZZER1.2
- no-connect marks 0 -> 1
