File: EMMC.kicad_sch (KiCad schematic)
At the start: 20 parts, among them U9 KLM8G1GETF-B0410

Commit message: 2026 08 24 画图完成，准备生产
Parts:
- C59, C60, C61, C62, C63: footprint Capacitor_SMD:C_0805_2012Metric_Pad1.18x1.45mm_HandSolder -> Capacitor_SMD:C_0603_1608Metric_Pad1.08x0.95mm_HandSolder
Connections:
- net GND: now also U9.C5 (NC_21), U9.N6 (NC_91), U9.P2 (NC_101)
- net Net-(U9A-CLK): now reaches R75.2, U9.M6 (CLK)
- net EMMC_VDDI: now reaches C58.1, U9.C2 (VDDI)
- net EMMC_VDDI: now also U9.C1 (NC_19)
- net EMMC_D3: now reaches R73.2, U9.B2 (DAT3)
- net EMMC_D3: now also U9.B1 (NC_10)
- net EMMC_D0: now reaches R74.2, U9.A3 (DAT0)
- net EMMC_D1: now reaches R71.2, U9.A4 (DAT1)
- net EMMC_D2: now reaches R72.2, U9.A5 (DAT2)
- no-connect marks 18 -> 120
