File: LCD.kicad_sch (KiCad schematic)
At the start: 47 parts, among them J1 Conn_01x50_MountingPin, U3 MP3302DJ-LF-P

Commit message: 2026 08 16 原理图完成，下一步制作分配未完成的器件封装，准备layout
Parts:
- removed R13: 4.7K, Resistor_SMD:R_0805_2012Metric_Pad1.20x1.40mm_HandSolder, symbol Device:R_US
- removed R14: 4.7K_NC, Resistor_SMD:R_0805_2012Metric_Pad1.20x1.40mm_HandSolder, symbol Device:R_US
- added C26, C27, C28, C29: 15pF, Capacitor_SMD:C_0603_1608Metric_Pad1.08x0.95mm_HandSolder, symbol Device:C
- added C33: 1uF, Capacitor_SMD:C_0603_1608Metric_Pad1.08x0.95mm_HandSolder, symbol Device:C
- added C34: 100nF, Capacitor_SMD:C_0603_1608Metric_Pad1.08x0.95mm_HandSolder, symbol Device:C
- added L2: CBG160808U121T, Inductor_SMD:L_0201_0603Metric_Pad0.64x0.40mm_HandSolder, symbol Device:L_Ferrite
- added R27: 4.7K, Resistor_SMD:R_0805_2012Metric_Pad1.20x1.40mm_HandSolder, symbol Device:R_US
- added R30: 4.7K_NC, Resistor_SMD:R_0805_2012Metric_Pad1.20x1.40mm_HandSolder, symbol Device:R_US
- added R35: 10K, Resistor_SMD:R_0603_1608Metric_Pad0.98x0.95mm_HandSolder, symbol Device:R_US
- added RN1, RN2, RN3, RN4, RN5: 22R X 4, Package_DIP:DIP-8-16_W7.62mm_Socket, symbol Device:R_Pack04
- added TP10: LCD_VDDA_TP, TestPoint:TestPoint_Pad_D3.0mm, symbol Connector:TestPoint
- added TP13: MP3302_SW_TP, TestPoint:TestPoint_Pad_D3.0mm, symbol Connector:TestPoint
- added TP14: LCD_CLK_TP, TestPoint:TestPoint_Pad_D3.0mm, symbol Connector:TestPoint
- added TP7: LCD_VGL_TP, TestPoint:TestPoint_Pad_D3.0mm, symbol Connector:TestPoint
- added TP8: LCD_VGH_TP, TestPoint:TestPoint_Pad_D3.0mm, symbol Connector:TestPoint
- added TP9: LCD_VCOM_TP, TestPoint:TestPoint_Pad_D3.0mm, symbol Connector:TestPoint
- J3: renamed from J1; footprint (none) -> Connector_FFC-FPC:Hirose_FH12-50S-0.5SH_1x50-1MP_P0.50mm_Horizontal
- L4: renamed from L2; footprint Inductor_SMD:L_Changjiang_FTC252010S -> Inductor_SMD:L_0603_1608Metric_Pad1.05x0.95mm_HandSolder
- gave numbers to parts that had none: 30
- renumbered C18 to C35, C16 to C36, C17 to C37, D4 to D10, R15 to R25, R17 to R26, R16 to R28, R18 to R29, R12 to R31, R19 to R32, R20 to R33, R11 to R34, U3 to U5
Connections:
- net DCLK: now also C29.1, L2.2
- net DE: now also C28.1, RN5.3 (R3.1)
- net GND: now also C26.2, C27.2, C28.2, C29.2, C33.2, C34.2, R30.2, R35.1
- net HSYNC: now also C27.1, RN5.2 (R2.1)
- net LCD_B0: now also RN1.4 (R4.1)
- net LCD_B1: now also RN1.3 (R3.1)
- net LCD_B2: now also RN1.2 (R2.1)
- net LCD_B3: now also RN1.1 (R1.1)
- net LCD_B4: now also RN2.4 (R4.1)
- net LCD_G0: now also RN2.3 (R3.1)
- net LCD_G1: now also RN2.2 (R2.1)
- net LCD_G2: now also RN2.1 (R1.1)
- net LCD_G3: now also RN3.4 (R4.1)
- net LCD_G4: now also RN3.3 (R3.1)
- net LCD_G5: now also RN3.2 (R2.1)
- net LCD_R0: now also RN3.1 (R1.1)
- net LCD_R1: now also RN4.4 (R4.1)
- net LCD_R2: now also RN4.3 (R3.1)
- net LCD_R3: now also RN4.2 (R2.1)
- net LCD_R4: now also RN4.1 (R1.1)
- net MODE: now also R27.2, R30.1
- net VCOM: now also TP9.1
- net VDD_A: now also TP10.1
- net VGH: now also TP8.1
- net VGL: now also TP7.1
- net VSYNC: now also C26.1, RN5.1 (R1.1)
- net at D10.2 (A), L4.2, U5.1 (SW): now also TP13.1
- net BLK renamed LCD_BLK
- net LCD_BLK: now also R35.2
- net VDD_D renamed LCD_3V3
- net LCD_3V3: now also C33.1, C34.1, R27.1
- net VIN_5V renamed LCD_VIN_5V
- new net: L2.1, RN5.4 (R4.1)
- new net LCDIF_CLK: RN5.5 (R4.2), TP14.1
- new net LCDIF_D0: RN1.5 (R4.2)
- new net LCDIF_D1: RN1.6 (R3.2)
- new net LCDIF_D10: RN3.7 (R2.2)
- new net LCDIF_D11: RN3.8 (R1.2)
- new net LCDIF_D12: RN4.5 (R4.2)
- new net LCDIF_D13: RN4.6 (R3.2)
- new net LCDIF_D14: RN4.7 (R2.2)
- new net LCDIF_D15: RN4.8 (R1.2)
- new net LCDIF_D2: RN1.7 (R2.2)
- new net LCDIF_D3: RN1.8 (R1.2)
- new net LCDIF_D4: RN2.5 (R4.2)
- new net LCDIF_D5: RN2.6 (R3.2)
- new net LCDIF_D6: RN2.7 (R2.2)
- new net LCDIF_D7: RN2.8 (R1.2)
- new net LCDIF_D8: RN3.5 (R4.2)
- new net LCDIF_D9: RN3.6 (R3.2)
- new net LCDIF_ENABLE: RN5.6 (R3.2)
- new net LCDIF_HSYNC: RN5.7 (R2.2)
- new net LCDIF_VSYNC: RN5.8 (R1.2)
Other:
- note added: "C17一定要靠近U3的PIN-5放置"
- moved on the sheet: C36, C37, J3, R25, R26, R28, R29, R34

Commit message: 2026 08 24 画图完成，准备生产
Parts:
- removed J3: Conn_01x50_MountingPin, Connector_FFC-FPC:Hirose_FH12-50S-0.5SH_1x50-1MP_P0.50mm_Horizontal, symbol Connector_Generic_MountingPin:Conn_01x50_MountingPin
- removed TP13: MP3302_SW_TP, TestPoint:TestPoint_Pad_D3.0mm, symbol Connector:TestPoint
- added J10: Conn_01x50_MountingPin, UPT:FPC-SMD_FH12A-50S-0.5SH-55-1, symbol Connector_Generic_MountingPin:Conn_01x50_MountingPin
- D10: value SS54 -> SS34
- L4: footprint Inductor_SMD:L_0603_1608Metric_Pad1.05x0.95mm_HandSolder -> Inductor_SMD:L_Changjiang_FTC252010S
- R20: footprint Resistor_SMD:R_1206_3216Metric_Pad1.30x1.75mm_HandSolder -> Resistor_SMD:R_0805_2012Metric_Pad1.20x1.40mm_HandSolder
- RN1, RN2, RN3, RN4, RN5: footprint Package_DIP:DIP-8-16_W7.62mm_Socket -> Resistor_SMD:R_Array_Concave_4x0603
- TP10, TP7, TP8, TP9: footprint TestPoint:TestPoint_Pad_D3.0mm -> TestPoint:TestPoint_Pad_D1.5mm
- TP14: footprint TestPoint:TestPoint_Pad_D3.0mm -> TestPoint:TestPoint_Pad_D1.0mm
- U4: footprint Package_DFN_QFN:VQFN-24-1EP_4x4mm_P0.5mm_EP2.45x2.45mm_ThermalVias -> Package_DFN_QFN:Texas_RGE0024H_VQFN-24-1EP_4x4mm_P0.5mm_EP2.7x2.7mm_ThermalVias
Connections:
- net DCLK: now also J10.14 (Pin_14)
- net DE: now also RN5.4 (R4.1), J10.42 (Pin_42); no longer RN5.3 (R3.1)
- net GND: now also J10.13 (Pin_13), J10.15 (Pin_15), J10.16 (Pin_16), J10.17 (Pin_17), J10.18 (Pin_18), J10.24 (Pin_24), J10.25 (Pin_25), J10.3 (Pin_3), J10.32 (Pin_32), J10.33 (Pin_33), J10.34 (Pin_34), J10.4 (Pin_4), J10.46 (Pin_46), J10.MP (MountPin)
- net HSYNC: now also C26.1, J10.40 (Pin_40); no longer C27.1
- net LCDIF_CLK: now also RN4.8 (R1.2); no longer RN5.5 (R4.2)
- net LCDIF_D0: now also RN1.8 (R1.2); no longer RN1.5 (R4.2)
- net LCDIF_D1: now also RN1.7 (R2.2); no longer RN1.6 (R3.2)
- net LCDIF_D10: now also RN3.5 (R4.2); no longer RN3.7 (R2.2)
- net LCDIF_D11: now also RN4.7 (R2.2); no longer RN3.8 (R1.2)
- net LCDIF_D12: now also RN4.6 (R3.2); no longer RN4.5 (R4.2)
- net LCDIF_D13: now also RN4.5 (R4.2); no longer RN4.6 (R3.2)
- net LCDIF_D14: now also RN2.8 (R1.2); no longer RN4.7 (R2.2)
- net LCDIF_D15: now also RN2.7 (R2.2); no longer RN4.8 (R1.2)
- net LCDIF_D2: now also RN1.6 (R3.2); no longer RN1.7 (R2.2)
- net LCDIF_D3: now also RN1.5 (R4.2); no longer RN1.8 (R1.2)
- net LCDIF_D4: now also RN5.8 (R1.2); no longer RN2.5 (R4.2)
- net LCDIF_D6: now also RN2.5 (R4.2); no longer RN2.7 (R2.2)
- net LCDIF_D7: now also RN3.8 (R1.2); no longer RN2.8 (R1.2)
- net LCDIF_D8: now also RN3.7 (R2.2); no longer RN3.5 (R4.2)
- net LCDIF_ENABLE: now also RN5.5 (R4.2); no longer RN5.6 (R3.2)
- net LCDIF_VSYNC: now also RN5.6 (R3.2); no longer RN5.8 (R1.2)
- net LCD_3V3: now also J10.44 (Pin_44)
- net LCD_B0: now also RN1.1 (R1.1), J10.35 (Pin_35); no longer RN1.4 (R4.1)
- net LCD_B1: now also RN1.2 (R2.1), J10.36 (Pin_36); no longer RN1.3 (R3.1)
- net LCD_B2: now also RN1.3 (R3.1), J10.37 (Pin_37); no longer RN1.2 (R2.1)
- net LCD_B3: now also RN1.4 (R4.1), J10.38 (Pin_38); no longer RN1.1 (R1.1)
- net LCD_B4: now also RN5.1 (R1.1), J10.39 (Pin_39); no longer RN2.4 (R4.1)
- net LCD_G0: now also J10.26 (Pin_26)
- net LCD_G1: now also RN2.4 (R4.1), J10.27 (Pin_27); no longer RN2.2 (R2.1)
- net LCD_G2: now also RN3.1 (R1.1), J10.28 (Pin_28); no longer RN2.1 (R1.1)
- net LCD_G3: now also RN3.2 (R2.1), J10.29 (Pin_29); no longer RN3.4 (R4.1)
- net LCD_G4: now also J10.30 (Pin_30)
- net LCD_G5: now also RN3.4 (R4.1), J10.31 (Pin_31); no longer RN3.2 (R2.1)
- net LCD_R0: now also RN4.2 (R2.1), J10.19 (Pin_19); no longer RN3.1 (R1.1)
- net LCD_R1: now also RN4.3 (R3.1), J10.20 (Pin_20); no longer RN4.4 (R4.1)
- net LCD_R2: now also RN4.4 (R4.1), J10.21 (Pin_21); no longer RN4.3 (R3.1)
- net LCD_R3: now also RN2.1 (R1.1), J10.22 (Pin_22); no longer RN4.2 (R2.1)
- net LCD_R4: now also RN2.2 (R2.1), J10.23 (Pin_23); no longer RN4.1 (R1.1)
- net LED_A: now also J10.49 (Pin_49), J10.50 (Pin_50)
- net LED_K: now also J10.47 (Pin_47), J10.48 (Pin_48)
- net L/R: now also J10.12 (Pin_12)
- net MODE: now also J10.43 (Pin_43)
- net U/D: now also J10.11 (Pin_11)
- net VCOM: now also J10.45 (Pin_45), J10.5 (Pin_5)
- net VDD_A: now also J10.8 (Pin_8)
- net VGH: now also J10.10 (Pin_10)
- net VGL: now also J10.9 (Pin_9)
- net VSYNC: now also C27.1, RN5.3 (R3.1), J10.41 (Pin_41); no longer C26.1, RN5.1 (R1.1)
- net at L2.1: now also RN4.1 (R1.1); no longer RN5.4 (R4.1)
- new net LCD_RST: J10.7 (Pin_7)
Other:
- note added: "FPC线序对比参照引脚需要翻转，因为FPC端子位于屏幕后方"
- note removed: "50PIN FPC Connector,Bottom contact"
- moved on the sheet: C26, C27, C28, R27, R30, RN5
