File: Power.kicad_sch (KiCad schematic)
At the start: 39 parts, among them J2 USB_C_Receptacle_USB2.0_16P, J5 Barrel_Jack_MountingPin, Q1 PMOS, SW4 SW_Push_DPDT, U2 MP9447GL-P, U3 MP20051DQ-LF-Z

Commit message: 2026 08 16 原理图完成，下一步制作分配未完成的器件封装，准备layout
Parts:
- added BT1: BS-2450-3, Battery:BatteryHolder_Keystone_103_1x20mm, symbol Device:Battery_Cell
- added D15: BAV70, Package_TO_SOT_SMD:SOT-23, symbol Diode:BAV70
- added TP12: VBAT_TP, TestPoint:TestPoint_Pad_D3.0mm, symbol Connector:TestPoint
- added TP15, TP16, TP3: GND_TP, Connector_PinHeader_2.54mm:PinHeader_1x01_P2.54mm_Vertical, symbol Connector:TestPoint
- added TP4: TYPEC_5V_TP, TestPoint:TestPoint_Pad_D3.0mm, symbol Connector:TestPoint
- added TP6: DCIN_24V_TP, TestPoint:TestPoint_Pad_D3.0mm, symbol Connector:TestPoint
- C10: renamed from C7; footprint (none) -> Capacitor_SMD:C_1210_3225Metric_Pad1.33x2.70mm_HandSolder
- C11: footprint (none) -> Capacitor_SMD:C_0805_2012Metric_Pad1.18x1.45mm_HandSolder
- C12: renamed from C4; footprint (none) -> Capacitor_SMD:C_0805_2012Metric_Pad1.18x1.45mm_HandSolder
- C2: renamed from C5; footprint (none) -> Capacitor_SMD:C_0603_1608Metric_Pad1.08x0.95mm_HandSolder
- C3: renamed from C9; footprint (none) -> Capacitor_SMD:C_0603_1608Metric_Pad1.08x0.95mm_HandSolder
- C4: renamed from C10; footprint (none) -> Capacitor_SMD:C_0805_2012Metric_Pad1.18x1.45mm_HandSolder
- C5: renamed from C1; footprint (none) -> Capacitor_SMD:C_1206_3216Metric_Pad1.33x1.80mm_HandSolder
- C6: renamed from C2; footprint (none) -> Capacitor_SMD:C_0603_1608Metric_Pad1.08x0.95mm_HandSolder
- C7: renamed from C3; footprint (none) -> Capacitor_SMD:C_0603_1608Metric_Pad1.08x0.95mm_HandSolder
- C8: footprint (none) -> Capacitor_SMD:C_0603_1608Metric_Pad1.08x0.95mm_HandSolder
- C9: renamed from C6; footprint (none) -> Capacitor_SMD:C_1210_3225Metric_Pad1.33x2.70mm_HandSolder
- D3: renamed from D2; footprint (none) -> Diode_SMD:D_SMB_Handsoldering
- D4: renamed from D3; footprint SOT95P230X110-3N -> UPT:SOT95P230X110-3N
- D5: renamed from D1; footprint (none) -> Capacitor_SMD:C_0805_2012Metric_Pad1.18x1.45mm_HandSolder
- D6: renamed from D5; footprint (none) -> Diode_SMD:D_SMA_Handsoldering
- F1: footprint (none) -> Fuse:Fuse_1206_3216Metric
- F2: footprint (none) -> Fuse:Fuse_1812_4532Metric
- J1: renamed from J2; footprint (none) -> Connector_USB:USB_C_Receptacle_GCT_USB4105-xx-A_16P_TopMnt_Horizontal
- L1: footprint (none) -> Inductor_SMD:L_APV_APH0630
- R10: renamed from R21; footprint (none) -> Resistor_SMD:R_0603_1608Metric_Pad0.98x0.95mm_HandSolder
- R11: renamed from R2; footprint (none) -> Resistor_SMD:R_0603_1608Metric_Pad0.98x0.95mm_HandSolder
- R12: renamed from R5; value 100K -> 10K; footprint (none) -> Resistor_SMD:R_0603_1608Metric_Pad0.98x0.95mm_HandSolder
- R13: renamed from R10; footprint (none) -> Resistor_SMD:R_0603_1608Metric_Pad0.98x0.95mm_HandSolder
- R14: renamed from R9; footprint (none) -> Resistor_SMD:R_0603_1608Metric_Pad0.98x0.95mm_HandSolder
- R15: renamed from R8; footprint (none) -> Resistor_SMD:R_0603_1608Metric_Pad0.98x0.95mm_HandSolder
- R4: renamed from R3; footprint (none) -> Resistor_SMD:R_0603_1608Metric_Pad0.98x0.95mm_HandSolder
- R5: renamed from R6; footprint (none) -> Resistor_SMD:R_0603_1608Metric_Pad0.98x0.95mm_HandSolder
- R6: renamed from R1; footprint (none) -> Resistor_SMD:R_0603_1608Metric_Pad0.98x0.95mm_HandSolder
- R7: renamed from R4; value 100K -> 53.6K; footprint (none) -> Capacitor_SMD:C_0603_1608Metric_Pad1.08x0.95mm_HandSolder
- R8: renamed from R4; footprint (none) -> Resistor_SMD:R_0603_1608Metric_Pad0.98x0.95mm_HandSolder
- R9: renamed from R7; footprint (none) -> Resistor_SMD:R_0603_1608Metric_Pad0.98x0.95mm_HandSolder
- TP1: renamed from TP3; footprint (none) -> Connector_PinHeader_2.54mm:PinHeader_1x01_P2.54mm_Vertical
- TP2: renamed from TP1; footprint (none) -> TestPoint:TestPoint_Pad_D3.0mm
- TP5: renamed from TP2; footprint (none) -> Connector_PinHeader_2.54mm:PinHeader_1x01_P2.54mm_Vertical
- U2: renamed from U3; footprint SON65P300X300X100-9N-D -> UPT:SON65P300X300X100-9N-D
- U3: renamed from U2; footprint MP9447GLP -> UPT:MP9447GLP
- renumbered J5 to J2, SW4 to SW1
Connections:
- net BASE_3V3: now also D15.2 (A)
- net DCDC_5V: now also TP4.1
- net DCIN_24V: now also TP6.1
- net GND: now also BT1.2 (-), TP15.1, TP16.1, TP3.1
- new net: BT1.1 (+), D15.1 (A), TP12.1
- new net COIN_BAT_3V3: D15.3 (K)
Other:
- note added: "BAT For RT1052_SNVS Power"
- note added: "MHCB06030-100M-C1"
- moved on the sheet: C4, TP5

Commit message: 2026 08 24 画图完成，准备生产
Parts:
- removed J2: Barrel_Jack_MountingPin, Connector_BarrelJack:BarrelJack_CUI_PJ-063AH_Horizontal, symbol Connector:Barrel_Jack_MountingPin
- added C85: 33nF, Capacitor_SMD:C_0603_1608Metric_Pad1.08x0.95mm_HandSolder, symbol Device:C
- added J2: DC-044A-A200, UPT:DC-IN-TH_DC-044A-20A, symbol Connector:Barrel_Jack_Switch_MountingPin
- BT1: footprint Battery:BatteryHolder_Keystone_103_1x20mm -> UPT:BAT-TH_BS-24-A1AJ013
- C6, C7: footprint Capacitor_SMD:C_0603_1608Metric_Pad1.08x0.95mm_HandSolder -> Capacitor_SMD:C_0805_2012Metric_Pad1.18x1.45mm_HandSolder
- Q1: value PMOS -> AO3401A; footprint (none) -> Package_TO_SOT_SMD:TSOT-23_HandSoldering
- SW1: footprint Button_Switch_THT:SW_PUSH_E-Switch_FS5700DP_DPDT -> UPT:SW-TH_5.8ZSGT
- TP12, TP2, TP4: footprint TestPoint:TestPoint_Pad_D3.0mm -> TestPoint:TestPoint_Pad_D1.5mm
Connections:
- net GND: now also C85.2, J2.2, J2.3, J2.MP (MountPin); no longer U3.4 (SS)
- net at SW1.2 (B), SW1.5 (B): now also J2.1
- new net: C85.1, U3.4 (SS)
Other:
- moved on the sheet: D5, R15, TP1
