File: USB.kicad_sch (KiCad schematic)
At the start: 7 parts, among them J3 USB_C_Receptacle_USB2.0_16P, U5 USBLC6-2SC6

Commit message: 2026 08 16 原理图完成，下一步制作分配未完成的器件封装，准备layout
Parts:
- J4: renamed from J3; footprint (none) -> Connector_USB:USB_C_Receptacle_GCT_USB4105-xx-A_16P_TopMnt_Horizontal
- L5: renamed from L3; value 600R,1A -> 600 Ohm @ 100MHz,1A
- R36: renamed from R22; footprint (none) -> Capacitor_SMD:C_0603_1608Metric_Pad1.08x0.95mm_HandSolder
- R37: renamed from R23; footprint (none) -> Capacitor_SMD:C_0603_1608Metric_Pad1.08x0.95mm_HandSolder
- renumbered D6 to D11, U5 to U6
Changed lines of the file:
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@@
 	(text "USB_OTG1_DEVICE\n"
 		(exclude_from_sim no)
-		(at 68.326 41.402 0)
+		(at 68.58 41.402 0)
 		(effects
 			(font
-				(face "Maple Mono NF Medium")
+				(face "KiCad Font")
 				(size 2.54 2.54)
-				(thickness 0.762)
-				(bold yes)
+				(thickness 0.3175)
 				(color 255 88 5 1)
 			)
@@
 		(color 0 0 0 0)
 	)
+	(junction
+		(at 154.94 71.12)
+		(diameter 0)
+		(color 0 0 0 0)
+	)
 	(no_connect
 		(at 113.03 99.06)
@@
 		(pts
 			(xy 152.4 86.36) (xy 168.91 86.36)
+		)
+		(stroke
+			(width 0)
+			(type default)
+		)
+	)
+	(wire
+		(pts
+			(xy 154.94 71.12) (xy 162.56 71.12)
 		)
 		(stroke
@@
 		(shape bidirectional)
 		(at 191.77 91.44 0)
+		(effects
+			(font
+				(size 1.27 1.27)
+			)
+			(justify left)
+		)
+	)
+	(hierarchical_label "USB_OTG1_VBUS"
+		(shape output)
+		(at 162.56 71.12 0)
 		(effects
 			(font
@@
 		(in_pos_files yes)
 		(dnp no)
-		(property "Reference" "#PWR053"
+		(property "Reference" "#PWR097"
 			(at 154.94 68.58 0)
 			(hide yes)
@@
 			(project "UWB_Positioning_Terminal"
 				(path "/b9bb75c4-3ddc-4c63-9df8-68118c9082ef/7163e9df-074e-4c31-a360-732920c23810"
-					(reference "#PWR053")
+					(reference "#PWR097")
 					(unit 1)
 				)
@@
 		(in_pos_files yes)
 		(dnp no)
-		(property "Reference" "R23"
+		(property "Reference" "R37"
 			(at 126.746 77.724 90)
 			(show_name no)
@@
 			)
 		)
-		(property "Footprint" ""
+		(property "Footprint" "Capacitor_SMD:C_0603_1608Metric_Pad1.08x0.95mm_HandSolder"
 			(at 133.604 77.724 90)
 			(hide yes)
@@
 			(project "UWB_Positioning_Terminal"
 				(path "/b9bb75c4-3ddc-4c63-9df8-68118c9082ef/7163e9df-074e-4c31-a360-732920c23810"
-					(reference "R23")
+					(reference "R37")
 					(unit 1)
 				)
@@
 		(in_pos_files yes)
 		(dnp no)
-		(property "Reference" "U5"
+		(property "Reference" "U6"
 			(at 174.752 95.504 0)
 			(show_name no)
@@
 			(project "UWB_Positioning_Terminal"
 				(path "/b9bb75c4-3ddc-4c63-9df8-68118c9082ef/7163e9df-074e-4c31-a360-732920c23810"
-					(reference "U5")
+					(reference "U6")
 					(unit 1)
 				)
@@
 		(in_pos_files yes)
 		(dnp no)
-		(property "Reference" "L3"
+		(property "Reference" "L5"
 			(at 121.92 70.104 90)
 			(show_name no)
@@
 			)
 		)
-		(property "Value" "600R,1A"
-			(at 128.27 67.31 90)
+		(property "Value" "600 Ohm @ 100MHz,1A"
+			(at 124.206 68.326 90)
 			(show_name no)
 			(do_not_autoplace no)
@@
 			(project "UWB_Positioning_Terminal"
 				(path "/b9bb75c4-3ddc-4c63-9df8-68118c9082ef/7163e9df-074e-4c31-a360-732920c23810"
-					(reference "L3")
+					(reference "L5")
 					(unit 1)
 				)
@@
 		(dnp no)
 		(fields_autoplaced yes)
-		(property "Reference" "D6"
+		(property "Reference" "D11"
 			(at 146.3675 64.77 0)
 			(show_name no)
@@
 			(project "UWB_Positioning_Terminal"
 				(path "/b9bb75c4-3ddc-4c63-9df8-68118c9082ef/7163e9df-074e-4c31-a360-732920c23810"
-					(reference "D6")
+					(reference "D11")
 					(unit 1)
 				)
@@
 		(dnp no)
 		(fields_autoplaced yes)
-		(property "Reference" "#PWR048"
+		(property "Reference" "#PWR0101"
 			(at 90.17 124.46 0)
 			(hide yes)
@@
 			(project "UWB_Positioning_Terminal"
 				(path "/b9bb75c4-3ddc-4c63-9df8-68118c9082ef/7163e9df-074e-4c31-a360-732920c23810"
-					(reference "#PWR048")
+					(reference "#PWR0101")
 					(unit 1)
 				)
@@
 		(in_pos_files yes)
 		(dnp no)
-		(property "Reference" "J3"
+		(property "Reference" "J4"
 			(at 81.534 67.31 0)
 			(show_name no)
@@
 			)
 		)
-		(property "Footprint" ""
+		(property "Footprint" "Connector_USB:USB_C_Receptacle_GCT_USB4105-xx-A_16P_TopMnt_Horizontal"
 			(at 101.6 86.36 0)
 			(hide yes)
@@
 			(project "UWB_Positioning_Terminal"
 				(path "/b9bb75c4-3ddc-4c63-9df8-68118c9082ef/7163e9df-074e-4c31-a360-732920c23810"
-					(reference "J3")
+					(reference "J4")
 					(unit 1)
 				)
@@
 		(in_pos_files yes)
 		(dnp no)
-		(property "Reference" "#PWR052"
+		(property "Reference" "#PWR099"
 			(at 179.07 86.36 0)
 			(hide yes)
@@
 			(project "UWB_Positioning_Terminal"
 				(path "/b9bb75c4-3ddc-4c63-9df8-68118c9082ef/7163e9df-074e-4c31-a360-732920c23810"
-					(reference "#PWR052")
+					(reference "#PWR099")
 					(unit 1)
 				)
@@
 		(in_pos_files yes)
 		(dnp no)
-		(property "Reference" "#PWR051"
+		(property "Reference" "#PWR0100"
 			(at 179.07 106.68 0)
 			(hide yes)
@@
 			(project "UWB_Positioning_Terminal"
 				(path "/b9bb75c4-3ddc-4c63-9df8-68118c9082ef/7163e9df-074e-4c31-a360-732920c23810"
-					(reference "#PWR051")
+					(reference "#PWR0100")
 					(unit 1)
 				)
@@
 		(in_pos_files yes)
 		(dnp no)
-		(property "Reference" "#PWR049"
+		(property "Reference" "#PWR098"
 			(at 147.32 87.63 0)
 			(hide yes)
@@
 			(project "UWB_Positioning_Terminal"
 				(path "/b9bb75c4-3ddc-4c63-9df8-68118c9082ef/7163e9df-074e-4c31-a360-732920c23810"
-					(reference "#PWR049")
+					(reference "#PWR098")
 					(unit 1)
 				)
@@
 		(in_pos_files yes)
 		(dnp no)
-		(property "Reference" "R22"
+		(property "Reference" "R36"
 			(at 126.746 75.184 90)
 			(show_name no)
@@
 			)
 		)
-		(property "Footprint" ""
+		(property "Footprint" "Capacitor_SMD:C_0603_1608Metric_Pad1.08x0.95mm_HandSolder"
 			(at 133.096 77.216 90)
 			(hide yes)
@@
 			(project "UWB_Positioning_Terminal"
 				(path "/b9bb75c4-3ddc-4c63-9df8-68118c9082ef/7163e9df-074e-4c31-a360-732920c23810"
-					(reference "R22")
+					(reference "R36")
 					(unit 1)
 				)
@@
 		(in_pos_files yes)
 		(dnp no)
-		(property "Reference" "#PWR050"
+		(property "Reference" "#PWR096"
 			(at 137.16 68.58 0)
 			(hide yes)
@@
 			(project "UWB_Positioning_Terminal"
 				(path "/b9bb75c4-3ddc-4c63-9df8-68118c9082ef/7163e9df-074e-4c31-a360-732920c23810"
-					(reference "#PWR050")
+					(reference "#PWR096")
 					(unit 1)
 				)

Commit message: 2026 08 24 画图完成，准备生产
Parts:
- FL1: footprint (none) -> UPT:DLW21SN121HQ2L
- L5: value 600 Ohm @ 100MHz,1A -> 600 Ohm @ 100MHz,MPZ2012S601AT000; footprint (none) -> Inductor_SMD:L_0805_2012Metric_Pad1.05x1.20mm_HandSolder
Connections:
- net USB_OTG1_DN: now also FL1.3; no longer U6.6 (I/O1)
- net USB_OTG1_DP: now also FL1.1; no longer U6.4 (I/O2)
- net USB_DEVICE_P: now reaches U6.3 (I/O2)
- net USB_DEVICE_P: now also J4.A6 (D+), J4.B6 (D+); no longer FL1.1
- net USB_DEVICE_N: now reaches U6.1 (I/O1)
- net USB_DEVICE_N: now also J4.A7 (D-), J4.B7 (D-); no longer FL1.3
- new net: FL1.2, U6.4 (I/O2)
- new net: FL1.4, U6.6 (I/O1)
Changed lines of the file:
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@@
+	(wire
+		(pts
+			(xy 203.2 93.98) (xy 224.79 93.98)
+		)
+		(stroke
+			(width 0)
+			(type default)
+		)
+	)
 	(wire
 		(pts
@@
 	(wire
 		(pts
-			(xy 152.4 86.36) (xy 168.91 86.36)
-		)
-		(stroke
-			(width 0)
-			(type default)
-		)
-	)
-	(wire
-		(pts
 			(xy 154.94 71.12) (xy 162.56 71.12)
 		)
@@
 	(wire
 		(pts
+			(xy 203.2 88.9) (xy 224.79 88.9)
+		)
+		(stroke
+			(width 0)
+			(type default)
+		)
+	)
+	(wire
+		(pts
 			(xy 127 88.9) (xy 127 91.44)
 		)
@@
 	(wire
 		(pts
-			(xy 127 91.44) (xy 142.24 91.44)
+			(xy 127 91.44) (xy 173.99 91.44)
 		)
 		(stroke
@@
 	(wire
 		(pts
-			(xy 184.15 91.44) (xy 191.77 91.44)
+			(xy 184.15 93.98) (xy 193.04 93.98)
 		)
 		(stroke
@@
 	(wire
 		(pts
-			(xy 152.4 91.44) (xy 173.99 91.44)
-		)
-		(stroke
-			(width 0)
-			(type default)
-		)
-	)
-	(wire
-		(pts
 			(xy 147.32 76.2) (xy 147.32 78.74)
 		)
@@
 	(wire
 		(pts
-			(xy 127 86.36) (xy 142.24 86.36)
+			(xy 127 86.36) (xy 168.91 86.36)
 		)
 		(stroke
@@
 	(wire
 		(pts
-			(xy 184.15 88.9) (xy 191.77 88.9)
+			(xy 184.15 88.9) (xy 193.04 88.9)
 		)
 		(stroke
@@
 	(wire
 		(pts
+			(xy 184.15 93.98) (xy 184.15 91.44)
+		)
+		(stroke
+			(width 0)
+			(type default)
+		)
+	)
+	(wire
+		(pts
 			(xy 168.91 88.9) (xy 173.99 88.9)
 		)
@@
 			(width 0)
 			(type default)
+		)
+	)
+	(label "USB_DEVICE_P"
+		(at 128.27 91.44 0)
+		(effects
+			(font
+				(size 1.27 1.27)
+			)
+			(justify left bottom)
+		)
+	)
+	(label "USB_DEVICE_N"
+		(at 128.27 86.36 0)
+		(effects
+			(font
+				(size 1.27 1.27)
+			)
+			(justify left bottom)
 		)
 	)
 	(hierarchical_label "USB_OTG1_DP"
 		(shape bidirectional)
-		(at 191.77 91.44 0)
+		(at 224.79 93.98 0)
 		(effects
 			(font
@@
 	(hierarchical_label "USB_OTG1_DN"
 		(shape bidirectional)
-		(at 191.77 88.9 0)
+		(at 224.79 88.9 0)
 		(effects
 			(font
@@
 			)
 			(justify left)
-		)
-	)
-	(symbol
-		(lib_id "Device:Filter_EMI_CommonMode")
-		(at 147.32 88.9 180)
-		(unit 1)
-		(body_style 1)
-		(exclude_from_sim no)
-		(in_bom yes)
-		(on_board yes)
-		(in_pos_files yes)
-		(dnp no)
-		(property "Reference" "FL1"
-			(at 143.51 92.71 0)
-			(show_name no)
-			(do_not_autoplace no)
-			(effects
-				(font
-					(size 1.27 1.27)
-				)
-			)
-		)
-		(property "Value" "DLW21SN900SQ2L"
-			(at 158.242 92.71 0)
-			(show_name no)
-			(do_not_autoplace no)
-			(effects
-				(font
-					(size 1.27 1.27)
-				)
-			)
-		)
-		(property "Footprint" ""
-			(at 147.32 89.916 0)
-			(hide yes)
-			(show_name no)
-			(do_not_autoplace no)
-			(effects
-				(font
-					(size 1.27 1.27)
-				)
-			)
-		)
-		(property "Datasheet" ""
-			(at 147.32 89.916 0)
-			(hide yes)
-			(show_name no)
-			(do_not_autoplace no)
-			(effects
-				(font
-					(size 1.27 1.27)
-				)
-			)
-		)
-		(property "Description" "EMI 2-inductor common mode filter"
-			(at 147.32 88.9 0)
-			(hide yes)
-			(show_name no)
-			(do_not_autoplace no)
-			(effects
-				(font
-					(size 1.27 1.27)
-				)
-			)
-		)
-		(pin "2"
-		)
-		(pin "3"
-		)
-		(pin "1"
-		)
-		(pin "4"
-		)
-		(instances
-			(project "UWB_Positioning_Terminal"
-				(path "/b9bb75c4-3ddc-4c63-9df8-68118c9082ef/7163e9df-074e-4c31-a360-732920c23810"
-					(reference "FL1")
-					(unit 1)
-				)
-			)
 		)
 	)
@@
 	)
 	(symbol
+		(lib_id "power:PWR_FLAG")
+		(at 137.16 71.12 180)
+		(unit 1)
+		(body_style 1)
+		(exclude_from_sim no)
+		(in_bom yes)
+		(on_board yes)
+		(in_pos_files yes)
+		(dnp no)
+		(property "Reference" "#FLG06"
+			(at 137.16 73.025 0)
+			(hide yes)
+			(show_name no)
+			(do_not_autoplace no)
+			(effects
+				(font
+					(size 1.27 1.27)
+				)
+			)
+		)
+		(property "Value" "PWR_FLAG"
+			(at 143.256 74.422 0)
+			(show_name no)
+			(do_not_autoplace no)
+			(effects
+				(font
+					(size 1.27 1.27)
+				)
+			)
+		)
+		(property "Footprint" ""
+			(at 137.16 71.12 0)
+			(hide yes)
+			(show_name no)
+			(do_not_autoplace no)
+			(effects
+				(font
+					(size 1.27 1.27)
+				)
+			)
+		)
+		(property "Datasheet" ""
+			(at 137.16 71.12 0)
+			(hide yes)
+			(show_name no)
+			(do_not_autoplace no)
+			(effects
+				(font
+					(size 1.27 1.27)
+				)
+			)
+		)
+		(property "Description" "Special symbol for telling ERC where power comes from"
+			(at 137.16 71.12 0)
+			(hide yes)
+			(show_name no)
+			(do_not_autoplace no)
+			(effects
+				(font
+					(size 1.27 1.27)
+				)
+			)
+		)
+		(pin "1"
+		)
+		(instances
+			(project "UWB_Positioning_Terminal"
+				(path "/b9bb75c4-3ddc-4c63-9df8-68118c9082ef/7163e9df-074e-4c31-a360-732920c23810"
+					(reference "#FLG06")
+					(unit 1)
+				)
+			)
+		)
+	)
+	(symbol
 		(lib_id "Device:R_US")
 		(at 133.35 78.74 90)
@@
 			)
 		)
-		(property "Value" "600 Ohm @ 100MHz,1A"
-			(at 124.206 68.326 90)
-			(show_name no)
-			(do_not_autoplace no)
-			(effects
-				(font
-					(size 1.27 1.27)
-				)
-			)
-		)
-		(property "Footprint" ""
+		(property "Value" "600 Ohm @ 100MHz,MPZ2012S601AT000"
+			(at 111.252 65.024 90)
+			(show_name no)
+			(do_not_autoplace no)
+			(effects
+				(font
+					(size 1.27 1.27)
+				)
+			)
+		)
+		(property "Footprint" "Inductor_SMD:L_0805_2012Metric_Pad1.05x1.20mm_HandSolder"
 			(at 128.27 71.12 0)
 			(hide yes)
@@
 					(unit 1)
 				)
+			)
+		)
+	)
+	(symbol
+		(lib_id "Device:Filter_EMI_CommonMode")
+		(at 198.12 91.44 180)
+		(unit 1)
+		(body_style 1)
+		(exclude_from_sim no)
+		(in_bom yes)
+		(on_board yes)
+		(in_pos_files yes)
+		(dnp no)
+		(property "Reference" "FL1"
+			(at 194.31 95.25 0)
+			(show_name no)
+			(do_not_autoplace no)
+			(effects
+				(font
+					(size 1.27 1.27)
+				)
+			)
+		)
+		(property "Value" "DLW21SN900SQ2L"
+			(at 209.042 95.25 0)
+			(show_name no)
+			(do_not_autoplace no)
+			(effects
+				(font
+					(size 1.27 1.27)
+				)
+			)
+		)
+		(property "Footprint" "UPT:DLW21SN121HQ2L"
+			(at 198.12 92.456 0)
+			(hide yes)
+			(show_name no)
+			(do_not_autoplace no)
+			(effects
+				(font
+					(size 1.27 1.27)
+				)
+			)
+		)
+		(property "Datasheet" ""
+			(at 198.12 92.456 0)
+			(hide yes)
+			(show_name no)
+			(do_not_autoplace no)
+			(effects
+				(font
+					(size 1.27 1.27)
+				)
+			)
+		)
+		(property "Description" "EMI 2-inductor common mode filter"
+			(at 198.12 91.44 0)
+			(hide yes)
+			(show_name no)
+			(do_not_autoplace no)
+			(effects
+				(font
+					(size 1.27 1.27)
+				)
+			)
+		)
+		(pin "2"
+		)
+		(pin "3"
+		)
+		(pin "1"
+		)
+		(pin "4"
+		)
+		(instances
+			(project "UWB_Positioning_Terminal"
+				(path "/b9bb75c4-3ddc-4c63-9df8-68118c9082ef/7163e9df-074e-4c31-a360-732920c23810"
+					(reference "FL1")
+					(unit 1)
+				)
